File: design/simple_4Mb.kicad_pcb (KiCad board)
At the start: 4 copper layers, 100 x 100 mm, 15 parts, among them U1 AS6C8008-55ZIN, U2 AS6C8008-55ZIN, U3 AS6C8008-55ZIN, U4 AS6C8008-55ZIN, U5 ATF22V10C-15PU

Commit message: Add datasheet for memory and production data
Other:
- board size 100 x 100 mm -> 78 x 100 mm
Changed lines of the file:
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@@
 	)
 	(gr_line
-		(start 200 150)
-		(end 200 50)
+		(start 198 150)
+		(end 198 50)
 		(stroke
 			(width 0.1)
@@
 	)
 	(gr_line
-		(start 100 50)
-		(end 200 50)
+		(start 124.993374 50.011848)
+		(end 198 50)
 		(stroke
 			(width 0.1)
@@
 	)
 	(gr_line
-		(start 100 150)
-		(end 200 150)
+		(start 125 150)
+		(end 198 150)
+		(stroke
+			(width 0.1)
+			(type default)
+		)
+		(layer "Edge.Cuts")
+	)
+	(gr_arc
+		(start 119.993374 55.011848)
+		(mid 121.45784 51.476314)
+		(end 124.993374 50.011848)
+		(stroke
+			(width 0.1)
+			(type default)
+		)
+		(layer "Edge.Cuts")
+	)
+	(gr_arc
+		(start 125 150)
+		(mid 121.464466 148.535534)
+		(end 120 145)
 		(stroke
 			(width 0.1)
@@
 	)
 	(gr_line
-		(start 120 50)
-		(end 120 150)
+		(start 119.993374 55.011848)
+		(end 120 145)
 		(stroke
 			(width 0.1)
@@
 	)
 	(gr_text "simple_4Mb RAM board for the rosco_m68k\nMalcolm Harrow, Feb 2025, v1\nhttps://github.com/harrowm/simple_4Mb.git"
-		(at 122.8 67.7 0)
+		(at 127.3 59.8 0)
 		(layer "F.SilkS")
 		(effects
